Commit message: scaled meshes and changed origin of hand_l and hand_r

File: Avatars/eric/urdf/avatar_eric.urdf (robot description, URDF)
Before this commit: robot avatar_eric, 87 links, 86 joints
Links:
- link hand_l: geometry visual mesh filename=package://iai_avatar_description/Avatars/eric/meshes_simple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 scale=0.01 0.01 0.01
- link hand_r: geometry visual mesh filename=package://iai_avatar_description/Avatars/eric/meshes_simple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 scale=0.01 0.01 0.01
- link head: geometry visual mesh filename=package://iai_avatar_description/Avatars/eric/meshes_simple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 scale=0.01 0.01 0.01
- link spine_03: geometry visual mesh filename=package://iai_avatar_description/Avatars/eric/meshes_simple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 scale=0.01 0.01 0.01
- link upperarm_l: geometry visual mesh filename=package://iai_avatar_description/Avatars/eric/meshes_simple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 scale=0.01 0.01 0.01
- link upperarm_r: geometry visual mesh filename=package://iai_avatar_description/Avatars/eric/meshes_simple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 scale=0.01 0.01 0.01
- link upperleg_l: geometry visual mesh filename=package://iai_avatar_description/Avatars/eric/meshes_simple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 scale=0.01 0.01 0.01
- link upperleg_r: geometry visual mesh filename=package://iai_avatar_description/Avatars/eric/meshes_simple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 scale=0.01 0.01 0.01

Commit message: updated urdf and owl to match rp_master skeleton

File: Avatars/eric/urdf/avatar_eric.urdf (robot description, URDF)
Before this commit: robot avatar_eric, 87 links, 86 joints
Links:
- removed link hip
- removed link lowerleg_l
- removed link lowerleg_r
- removed link lowerleg_twist_l
- removed link lowerleg_twist_r
- removed link neck
- removed link shoulder_l
- removed link shoulder_r
- removed link upperleg_l
- removed link upperleg_r
- removed link upperleg_twist_l
- removed link upperleg_twist_r
- added link calf_l
- added link calf_r
- added link calf_twist_l
- added link calf_twist_r
- added link clavicle_l
- added link clavicle_r
- added link neck_01
- added link pelvis
- added link thigh_l; visual mesh filename=package://iai_avatar_description/Avatars/eric/meshes_simple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 scale=0.01 0.01 0.01
- added link thigh_r; visual mesh filename=package://iai_avatar_description/Avatars/eric/meshes_simple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 scale=0.01 0.01 0.01
- added link thigh_twist_l
- added link thigh_twist_r
Joints:
- removed joint hip_to_spine_01
- removed joint hip_to_upperleg_l
- removed joint hip_to_upperleg_r
- removed joint lowerleg_l_to_foot_l
- removed joint lowerleg_l_to_lowerleg_twist_l
- removed joint lowerleg_r_to_foot_r
- removed joint lowerleg_r_to_lowerleg_twist_r
- removed joint neck_to_head
- removed joint root_to_hip
- removed joint shoulder_l_to_upperarm_l
- removed joint shoulder_r_to_upperarm_r
- removed joint spine_03_to_neck
- removed joint spine_03_to_shoulder_l
- removed joint spine_03_to_shoulder_r
- removed joint upperleg_l_to_lowerleg_l
- removed joint upperleg_l_to_upperleg_twist_l
- removed joint upperleg_r_to_lowerleg_r
- removed joint upperleg_r_to_upperleg_twist_r
- added joint calf_l_to_calf_twist_l: type fixed, parent calf_l, child calf_twist_l, origin xyz=-0.220735520124 0.0143435029313 -0.0151363778859 rpy=0.0241432338953 8.12411308289e-05 -0.00107330083847
- added joint calf_l_to_foot_l: type fixed, parent calf_l, child foot_l, origin xyz=-0.421743512154 0.0208540670574 -0.0276844631881 rpy=0.0182572603226 0.0458440929651 0.00348563492298
- added joint calf_r_to_calf_twist_r: type fixed, parent calf_r, child calf_twist_r, origin xyz=0.22137466073 -0.0116511350498 0.0148830814287 rpy=0.051498323679 0.000987589359283 -0.00231440365314
- added joint calf_r_to_foot_r: type fixed, parent calf_r, child foot_r, origin xyz=0.419454842806 -0.0155709739774 0.0269763749093 rpy=0.0545608997345 0.045284897089 0.169531449676
- added joint clavicle_l_to_upperarm_l: type fixed, parent clavicle_l, child upperarm_l, origin xyz=0.128845497966 0.0631972700357 -0.0019424300408 rpy=0.0238880813122 0.469722896814 -0.13654795289
- added joint clavicle_r_to_upperarm_r: type fixed, parent clavicle_r, child upperarm_r, origin xyz=-0.120959401131 -0.0593282207847 0.00182377407327 rpy=0.2090934515 0.451155275106 -0.327468305826
- added joint neck_01_to_head: type fixed, parent neck_01, child head, origin xyz=0.0755760595202 -0.00537412054837 -0.00097730034031 rpy=0.0681002438068 0.00491692125797 0.174194231629
- added joint pelvis_to_spine_01: type fixed, parent pelvis, child spine_01, origin xyz=0.147955521941 -0.0129172177985 -5.01933818953e-08 rpy=0.9887383711231866 0.0008396338430066877 0.01093147511109891
- added joint pelvis_to_thigh_l: type fixed, parent pelvis, child thigh_l, origin xyz=-0.0145145617425 -0.00518470583484 -0.0899454131722 rpy=0.140670761466 -0.0486810952425 0.172580957413
- added joint pelvis_to_thigh_r: type fixed, parent pelvis, child thigh_r, origin xyz=-0.0145128397271 -0.00518464576453 0.089945524931 rpy=-0.0224179774523 -0.0360192358494 -0.997545480728
- added joint root_to_pelvis: type fixed, parent root, child pelvis, origin xyz=-0.00327410455793 0.101470641792 0.9128947258 rpy=-0.008681337481024287 0.24583410449739423 0.2416461027967589
- added joint spine_03_to_clavicle_l: type fixed, parent spine_03, child clavicle_l, origin xyz=0.103866547346 -0.0124222813174 -0.0371810607612 rpy=0.0974436700344 0.725871682167 0.0150327533484
- added joint spine_03_to_clavicle_r: type fixed, parent spine_03, child clavicle_r, origin xyz=0.109931521118 -0.0129764638841 0.0294459741563 rpy=0.676524996758 -0.0702666938305 -0.732984602451
- added joint spine_03_to_neck_01: type fixed, parent spine_03, child neck_01, origin xyz=0.148433417082 0.0128616830334 -0.00602402957156 rpy=0.0797079652548 0.0167903900146 -0.04035808146
- added joint thigh_l_to_calf_l: type fixed, parent thigh_l, child calf_l, origin xyz=-0.420130312443 1.00386763791e-07 1.60618839118e-07 rpy=0.00360685586929 -0.0122226774693 -0.173642396927
- added joint thigh_l_to_thigh_twist_l: type fixed, parent thigh_l, child thigh_twist_l, origin xyz=-0.20844489336 0.00411380454898 -0.0257120840251 rpy=-0.0338423848152 -3.13520431519e-05 0.00150185823441
- added joint thigh_r_to_calf_r: type fixed, parent thigh_r, child calf_r, origin xyz=0.418992042542 8.03094195589e-08 -1.20464122233e-07 rpy=-0.0120081305504 -0.012731730938 -0.216187998652
- added joint thigh_r_to_thigh_twist_r: type fixed, parent thigh_r, child thigh_twist_r, origin xyz=0.207881107926 -0.00411987304688 0.0256331600249 rpy=0.0548547059298 0.000125348567963 -0.00242139399052

Commit message: changed scale of meshes to 1 1 1

File: Avatars/eric/urdf/avatar_eric.urdf (robot description, URDF)
Before this commit: robot avatar_eric, 87 links, 86 joints
Links:
- link hand_l: geometry visual mesh filename=package://iai_avatar_description/Avatars/eric/meshes_simple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 scale=1 1 1
- link hand_r: geometry visual mesh filename=package://iai_avatar_description/Avatars/eric/meshes_simple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 scale=1 1 1
- link head: geometry visual mesh filename=package://iai_avatar_description/Avatars/eric/meshes_simple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 scale=1 1 1
- link spine_03: geometry visual mesh filename=package://iai_avatar_description/Avatars/eric/meshes_simple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 scale=1 1 1
- link thigh_l: geometry visual mesh filename=package://iai_avatar_description/Avatars/eric/meshes_simple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 scale=1 1 1
- link thigh_r: geometry visual mesh filename=package://iai_avatar_description/Avatars/eric/meshes_simple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 scale=1 1 1
- link upperarm_l: geometry visual mesh filename=package://iai_avatar_description/Avatars/eric/meshes_simple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 scale=1 1 1
- link upperarm_r: geometry visual mesh filename=package://iai_avatar_description/Avatars/eric/meshes_simple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 scale=1 1 1
