Commit message: added new links and joints to urdf file

File: MetaHuman/pia/urdf/avatar_pia.urdf (robot description, URDF)
Before this commit: robot avatar_pia, 87 links, 86 joints
Links:
- added link neck_02
- added link spine_04; visual mesh filename=package://iai_avatar_description/MetaHuman/pia/meshes/torso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
- added link spine_05
- link hand_l: geometry visual mesh filename=package://iai_avatar_description/MetaHuman/pia/meshes/hand_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
- link hand_r: geometry visual mesh filename=package://iai_avatar_description/MetaHuman/pia/meshes/hand_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
- link head: geometry visual mesh filename=package://iai_avatar_description/MetaHuman/pia/meshes/head.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
- link pelvis: geometry visual mesh filename=package://iai_avatar_description/MetaHuman/pia/meshes/legs.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
- link root: geometry visual mesh filename=package://iai_avatar_description/MetaHuman/pia/meshes/feet.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
- link spine_03: geometry 
- link thigh_l: geometry 
- link thigh_r: geometry 
- link upperarm_l: geometry 
- link upperarm_r: geometry 
Joints:
- removed joint neck_01_to_head
- removed joint spine_03_to_neck_01
- added joint neck_01_to_neck_02: type fixed, parent neck_01, child neck_02, origin xyz=0.0755760595202 -0.00537412054837 -0.00097730034031 rpy=0.0681002438068 0.00491692125797 0.174194231629
- added joint neck_02_to_head: type fixed, parent neck_02, child head, origin xyz=0.0755760595202 -0.00537412054837 -0.00097730034031 rpy=0.0681002438068 0.00491692125797 0.174194231629
- added joint spine_03_to_spine_04: type fixed, parent spine_03, child spine_04, origin xyz=0.148433417082 0.0128616830334 -0.00602402957156 rpy=0.0797079652548 0.0167903900146 -0.04035808146
- added joint spine_04_to_spine_05: type fixed, parent spine_04, child spine_05, origin xyz=0.0755760595202 -0.00537412054837 -0.00097730034031 rpy=0.0681002438068 0.00491692125797 0.174194231629
- added joint spine_05_to_neck_01: type fixed, parent spine_05, child neck_01, origin xyz=0.0755760595202 -0.00537412054837 -0.00097730034031 rpy=0.0681002438068 0.00491692125797 0.174194231629

Commit message: updated urdf file

File: MetaHuman/pia/urdf/avatar_pia.urdf (robot description, URDF)
Before this commit: robot avatar_pia, 90 links, 89 joints
Links:
- removed link calf_twist_l
- removed link calf_twist_r
- removed link eye_end_l
- removed link eye_end_r
- removed link foot_end_l
- removed link foot_end_r
- removed link head_end
- removed link ik_foot_l
- removed link ik_foot_r
- removed link ik_foot_root
- removed link ik_hand_gun
- removed link ik_hand_l
- removed link ik_hand_r
- removed link ik_hand_root
- removed link index_end_l
- removed link index_end_r
- removed link jaw_end
- removed link lowerarm_twist_l
- removed link lowerarm_twist_r
- removed link middle_end_l
- removed link middle_end_r
- removed link pinky_end_l
- removed link pinky_end_r
- removed link ring_end_l
- removed link ring_end_r
- removed link thigh_twist_l
- removed link thigh_twist_r
- removed link thumb_end_l
- removed link thumb_end_r
- removed link upperarm_twist_l
- removed link upperarm_twist_r
Joints:
- removed joint ball_l_to_foot_end_l
- removed joint ball_r_to_foot_end_r
- removed joint calf_l_to_calf_twist_l
- removed joint calf_r_to_calf_twist_r
- removed joint eye_l_to_eye_end_l
- removed joint eye_r_to_eye_end_r
- removed joint head_to_head_end
- removed joint ik_foot_root_to_ik_foot_l
- removed joint ik_foot_root_to_ik_foot_r
- removed joint ik_hand_gun_to_ik_hand_l
- removed joint ik_hand_gun_to_ik_hand_r
- removed joint ik_hand_root_to_ik_hand_gun
- removed joint index_03_l_to_index_end_l
- removed joint index_03_r_to_index_end_r
- removed joint jaw_to_jaw_end
- removed joint lowerarm_l_to_lowerarm_twist_l
- removed joint lowerarm_r_to_lowerarm_twist_r
- removed joint middle_03_l_to_middle_end_l
- removed joint middle_03_r_to_middle_end_r
- removed joint pinky_03_l_to_pinky_end_l
- removed joint pinky_03_r_to_pinky_end_r
- removed joint ring_03_l_to_ring_end_l
- removed joint ring_03_r_to_ring_end_r
- removed joint root_to_ik_foot_root
- removed joint root_to_ik_hand_root
- removed joint thigh_l_to_thigh_twist_l
- removed joint thigh_r_to_thigh_twist_r
- removed joint thumb_03_l_to_thumb_end_l
- removed joint thumb_03_r_to_thumb_end_r
- removed joint upperarm_l_to_upperarm_twist_l
- removed joint upperarm_r_to_upperarm_twist_r
- joint pelvis_to_thigh_l: type fixed -> continuous

Commit message: updated urdf file

File: MetaHuman/pia/urdf/avatar_pia.urdf (robot description, URDF)
Before this commit: robot avatar_pia, 59 links, 58 joints
Links:
- link calf_l: geometry visual mesh filename=package://iai_avatar_description/MetaHuman/pia/meshes/calf_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
- link calf_r: geometry visual mesh filename=package://iai_avatar_description/MetaHuman/pia/meshes/calf_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
- link foot_l: geometry visual mesh filename=package://iai_avatar_description/MetaHuman/pia/meshes/foot_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
- link foot_r: geometry visual mesh filename=package://iai_avatar_description/MetaHuman/pia/meshes/foot_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
- link lowerarm_l: geometry visual mesh filename=package://iai_avatar_description/MetaHuman/pia/meshes/lower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
- link lowerarm_r: geometry visual mesh filename=package://iai_avatar_description/MetaHuman/pia/meshes/lower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
- link pelvis: geometry visual mesh filename=package://iai_avatar_description/MetaHuman/pia/meshes/hip.o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
- link root: geometry 
- link spine_03: geometry visual mesh filename=package://iai_avatar_description/MetaHuman/pia/meshes/torso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
- link spine_04: geometry 
- link thigh_l: geometry visual mesh filename=package://iai_avatar_description/MetaHuman/pia/meshes/thigh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
- link thigh_r: geometry visual mesh filename=package://iai_avatar_description/MetaHuman/pia/meshes/thigh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
- link upperarm_l: geometry visual mesh filename=package://iai_avatar_description/MetaHuman/pia/meshes/upper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
- link upperarm_r: geometry visual mesh filename=package://iai_avatar_description/MetaHuman/pia/meshes/upper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
Joints:
- joint pelvis_to_thigh_l: type continuous -> fixed
